Commit message: Added EE params. Working now.

File: controller/urdf/alternative_dyn_params.xacro (robot description, xacro)
@@ -1,5 +1,5 @@
 <?xml version="1.0" encoding="utf-8" ?>
 <robot xmlns:xacro="http://www.ros.org/wiki/xacro" name="hand">
-    <xacro:property name="dyn_param_link0">
+    <xacro:property name="dyn_param_link1">
         <inertial>
             <origin rpy="0 0 0" xyz="-0.003875 0.002081 0.0" />
@@ -8,5 +8,5 @@
         </inertial>
     </xacro:property>
-    <xacro:property name="dyn_param_link1">
+    <xacro:property name="dyn_param_link2">
         <inertial>
             <origin rpy="0 0 0" xyz="-3.141e-03 -2.872e-02 3.495e-03" />
@@ -15,5 +15,5 @@
         </inertial>
     </xacro:property>
-    <xacro:property name="dyn_param_link2">
+    <xacro:property name="dyn_param_link3">
         <inertial>
             <origin rpy="0 0 0" xyz="2.7518e-02 3.9252e-02 -6.6502e-02" />
@@ -22,5 +22,5 @@
         </inertial>
     </xacro:property>
-    <xacro:property name="dyn_param_link3">
+    <xacro:property name="dyn_param_link4">
         <inertial>
             <origin rpy="0 0 0" xyz="-5.317e-02 1.04419e-01 2.7454e-02" />
@@ -29,5 +29,5 @@
         </inertial>
     </xacro:property>
-    <xacro:property name="dyn_param_link4">
+    <xacro:property name="dyn_param_link5">
         <inertial>
             <origin rpy="0 0 0" xyz="-1.1953e-02 4.1065e-02 -3.8437e-02" />
@@ -36,5 +36,5 @@
         </inertial>
     </xacro:property>
-    <xacro:property name="dyn_param_link5">
+    <xacro:property name="dyn_param_link6">
         <inertial>
             <origin rpy="0 0 0" xyz="6.0149e-02 -1.4117e-02 -1.0517e-02" />
@@ -43,5 +43,5 @@
         </inertial>
     </xacro:property>
-    <xacro:property name="dyn_param_link6">
+    <xacro:property name="dyn_param_link7">
         <inertial>
             <origin rpy="0 0 0" xyz="1.0517e-02 -4.252e-03 6.1597e-02" />
@@ -50,3 +50,10 @@
         </inertial>
     </xacro:property>
+    <xacro:property name="dyn_param_panda_hand">
+        <inertial>
+            <origin rpy="0 0 0" xyz="0.0 0.0 0.1034" />
+            <mass value="0.73" />
+            <inertia ixx="0.001" ixy="0.0" ixz="0.0" iyy="0.0025" iyz="0.0" izz="0.0017" />
+        </inertial>
+    </xacro:property>
 </robot>

File: controller/urdf/panda_arm.xacro (robot description, xacro)
@@ -20,7 +20,4 @@
         </geometry>
       </collision>
-      <xacro:if value="${use_alt_dyn_params}">
-        <xacro:insert_block name="dyn_param_link0" />
-      </xacro:if>
     </link>
     <link name="${arm_id}_link1">
@@ -173,4 +170,7 @@
         </geometry>
       </collision>
+      <xacro:if value="${use_alt_dyn_params}">
+        <xacro:insert_block name="dyn_param_link7" />
+      </xacro:if>
     </link>
     <joint name="${arm_id}_joint7" type="revolute">
