Commit message: fix KDL dynamics code

File: panda_dynamics_model/urdf/alternative_dyn_params.xacro (robot description, xacro)
@@ -1,5 +1,5 @@
 <?xml version="1.0" encoding="utf-8" ?>
-<robot xmlns:xacro="http://www.ros.org/wiki/xacro" name="hand">
-    <xacro:property name="dyn_param_link1">
+<robot xmlns:xacro="http://www.ros.org/wiki/xacro" name="panda_dyn">
+    <xacro:property name="panda_link1">
         <inertial>
             <origin rpy="0 0 0" xyz="-0.003875 0.002081 0.0" />
@@ -8,5 +8,5 @@
         </inertial>
     </xacro:property>
-    <xacro:property name="dyn_param_link2">
+    <xacro:property name="panda_link2">
         <inertial>
             <origin rpy="0 0 0" xyz="-3.141e-03 -2.872e-02 3.495e-03" />
@@ -15,5 +15,5 @@
         </inertial>
     </xacro:property>
-    <xacro:property name="dyn_param_link3">
+    <xacro:property name="panda_link3">
         <inertial>
             <origin rpy="0 0 0" xyz="2.7518e-02 3.9252e-02 -6.6502e-02" />
@@ -22,5 +22,5 @@
         </inertial>
     </xacro:property>
-    <xacro:property name="dyn_param_link4">
+    <xacro:property name="panda_link4">
         <inertial>
             <origin rpy="0 0 0" xyz="-5.317e-02 1.04419e-01 2.7454e-02" />
@@ -29,5 +29,5 @@
         </inertial>
     </xacro:property>
-    <xacro:property name="dyn_param_link5">
+    <xacro:property name="panda_link5">
         <inertial>
             <origin rpy="0 0 0" xyz="-1.1953e-02 4.1065e-02 -3.8437e-02" />
@@ -36,5 +36,5 @@
         </inertial>
     </xacro:property>
-    <xacro:property name="dyn_param_link6">
+    <xacro:property name="panda_link6">
         <inertial>
             <origin rpy="0 0 0" xyz="6.0149e-02 -1.4117e-02 -1.0517e-02" />
@@ -43,5 +43,5 @@
         </inertial>
     </xacro:property>
-    <xacro:property name="dyn_param_link7">
+    <xacro:property name="panda_link7">
         <inertial>
             <origin rpy="0 0 0" xyz="1.0517e-02 -4.252e-03 6.1597e-02" />
@@ -50,5 +50,5 @@
         </inertial>
     </xacro:property>
-    <xacro:property name="dyn_param_panda_hand">
+    <xacro:property name="panda_hand">
         <inertial>
             <origin rpy="0 0 0" xyz="0.0 0.0 0.1034" />

File: panda_dynamics_model/urdf/panda_arm_alt_dyn.urdf.xacro (robot description, xacro)
@@ -2,4 +2,5 @@
 <robot xmlns:xacro="http://www.ros.org/wiki/xacro" name="panda">
   <xacro:property name="use_alt_dyn_params" value="True" />
-  <xacro:include filename="$(find panda_dynamics_model)/urdf/alternative_dyn_params.xacro" />
+  <xacro:include filename="$(find panda_dynamics_model)/urdf/panda_arm_plus_inertial.xacro" />
+  <xacro:panda_arm safety_distance="0.03"/>
 </robot>

File: panda_dynamics_model/urdf/panda_arm_hand_alt_dyn.urdf.xacro (robot description, xacro)
@@ -2,5 +2,6 @@
 <robot xmlns:xacro="http://www.ros.org/wiki/xacro" name="panda">
   <xacro:property name="use_alt_dyn_params" value="True" />
-  <xacro:include filename="$(find panda_dynamics_model)/urdf/alternative_dyn_params.xacro" />
-  <xacro:include filename="$(find franka_description)/robots/panda_arm_hand.urdf.xacro" />
+  <xacro:include filename="$(find panda_dynamics_model)/urdf/panda_arm_plus_inertial.xacro" />
+  <xacro:include filename="$(find franka_description)/robots/hand.xacro" />
+  <xacro:panda_arm safety_distance="0.03"/>
 </robot>
