Commit message: enable loading of multiple panda arms

File: panda_dynamics_model/urdf/panda_arm_hand.urdf.xacro (robot description, xacro)
@@ -1,5 +1,5 @@
 <?xml version="1.0" encoding="utf-8" ?>
-<robot xmlns:xacro="http://www.ros.org/wiki/xacro" name="panda">
-  <xacro:property name="use_alt_dyn_params" value="True" />
+<robot xmlns:xacro="http://www.ros.org/wiki/xacro" name="$(arg arm_id)">
+  <xacro:arg name="arm_id" default="$(arg arm_id)" />
   <xacro:include filename="$(find panda_dynamics_model)/urdf/panda_arm_plus_inertial.xacro" />
   <xacro:include filename="$(find franka_description)/robots/hand.xacro" />

File: panda_dynamics_model/urdf/panda_arm_plus_inertial.xacro (robot description, xacro)
@@ -1,7 +1,8 @@
 <?xml version='1.0' encoding='utf-8'?>
 <robot xmlns:xacro="http://www.ros.org/wiki/xacro" name="panda">
+  <xacro:arg name="arm_id" default="panda" />
   <!-- safety_distance: Minimum safety distance in [m] by which the collision volumes are expanded and which is enforced during robot motions -->
   <!-- arm_id: Namespace of the panda arm. Serves to differentiate between arms in case of multiple instances. -->
-  <xacro:macro name="panda_arm" params="arm_id:='panda' description_pkg:='franka_description' connected_to:='' xyz:='0 0 0' rpy:='0 0 0' safety_distance:=0">
+  <xacro:macro name="panda_arm" params="arm_id:='$(arg arm_id)' description_pkg:='franka_description' connected_to:='' xyz:='0 0 0' rpy:='0 0 0' safety_distance:=0">
     <xacro:unless value="${not connected_to}">
       <joint name="${arm_id}_joint_${connected_to}" type="fixed">
