Commit message: rename franka_description to franka_description_mti to avoid name clashes

File: franka_description/robots/dual_panda_example.urdf.xacro (robot description, xacro)
@@ -3,6 +3,6 @@
   <xacro:arg name="arm_id_1" default="panda_1" />
   <xacro:arg name="arm_id_2" default="panda_2" />
-  <xacro:include filename="$(find franka_description)/robots/panda_arm.xacro"/>
-  <xacro:include filename="$(find franka_description)/robots/hand.xacro"/>
+  <xacro:include filename="$(find franka_description_mti)/robots/panda_arm.xacro"/>
+  <xacro:include filename="$(find franka_description_mti)/robots/hand.xacro"/>
   <!-- box shaped table as base for the 2 Pandas -->
   <link name="base">

File: franka_description/robots/hand.xacro (robot description, xacro)
@@ -13,5 +13,5 @@
       <visual>
         <geometry>
-          <mesh filename="package://franka_description/meshes/visual/hand.dae"/>
+          <mesh filename="package://franka_description_mti/meshes/visual/hand.dae"/>
         </geometry>
       </visual>
@@ -56,5 +56,5 @@
       <visual>
         <geometry>
-          <mesh filename="package://franka_description/meshes/visual/finger.dae"/>
+          <mesh filename="package://franka_description_mti/meshes/visual/finger.dae"/>
         </geometry>
       </visual>
@@ -64,5 +64,5 @@
         <origin xyz="0 0 0" rpy="0 0 ${pi}"/>
         <geometry>
-          <mesh filename="package://franka_description/meshes/visual/finger.dae"/>
+          <mesh filename="package://franka_description_mti/meshes/visual/finger.dae"/>
         </geometry>
       </visual>

File: franka_description/robots/panda_arm.urdf.xacro (robot description, xacro)
@@ -1,5 +1,5 @@
 <?xml version='1.0' encoding='utf-8'?>
 <robot xmlns:xacro="http://www.ros.org/wiki/xacro" name="panda">
-  <xacro:include filename="$(find franka_description)/robots/panda_arm.xacro" />
+  <xacro:include filename="$(find franka_description_mti)/robots/panda_arm.xacro" />
   <xacro:panda_arm safety_distance="0.03"/>
 </robot>

File: franka_description/robots/panda_arm.xacro (robot description, xacro)
@@ -3,5 +3,5 @@
   <!-- safety_distance: Minimum safety distance in [m] by which the collision volumes are expanded and which is enforced during robot motions -->
   <!-- arm_id: Namespace of the panda arm. Serves to differentiate between arms in case of multiple instances. -->
-  <xacro:macro name="panda_arm" params="arm_id:='panda' description_pkg:='franka_description' connected_to:='' xyz:='0 0 0' rpy:='0 0 0' safety_distance:=0">
+  <xacro:macro name="panda_arm" params="arm_id:='panda' description_pkg:='franka_description_mti' connected_to:='' xyz:='0 0 0' rpy:='0 0 0' safety_distance:=0">
     <xacro:unless value="${not connected_to}">
       <joint name="${arm_id}_joint_${connected_to}" type="fixed">

File: franka_description/robots/panda_arm_hand.urdf.xacro (robot description, xacro)
@@ -1,6 +1,6 @@
 <?xml version="1.0" encoding="utf-8"?>
 <robot xmlns:xacro="http://www.ros.org/wiki/xacro" name="panda">
-  <xacro:include filename="$(find franka_description)/robots/panda_arm.xacro"/>
-  <xacro:include filename="$(find franka_description)/robots/hand.xacro"/>
+  <xacro:include filename="$(find franka_description_mti)/robots/panda_arm.xacro"/>
+  <xacro:include filename="$(find franka_description_mti)/robots/hand.xacro"/>
   <xacro:panda_arm safety_distance="0.03"/>
   <xacro:hand ns="panda" rpy="0 0 ${-pi/4}" connected_to="panda_link8" safety_distance="0.03"/>

File: panda_dynamics_model/urdf/panda_arm_hand.urdf.xacro (robot description, xacro)
@@ -3,5 +3,5 @@
   <xacro:arg name="arm_id" default="$(arg arm_id)" />
   <xacro:include filename="$(find panda_dynamics_model)/urdf/panda_arm_plus_inertial.xacro" />
-  <xacro:include filename="$(find franka_description)/robots/hand.xacro" />
+  <xacro:include filename="$(find franka_description_mti)/robots/hand.xacro" />
   <xacro:panda_arm safety_distance="0.03"/>
 </robot>

File: panda_dynamics_model/urdf/panda_arm_plus_inertial.xacro (robot description, xacro)
@@ -4,5 +4,5 @@
   <!-- safety_distance: Minimum safety distance in [m] by which the collision volumes are expanded and which is enforced during robot motions -->
   <!-- arm_id: Namespace of the panda arm. Serves to differentiate between arms in case of multiple instances. -->
-  <xacro:macro name="panda_arm" params="arm_id:='$(arg arm_id)' description_pkg:='franka_description' connected_to:='' xyz:='0 0 0' rpy:='0 0 0' safety_distance:=0">
+  <xacro:macro name="panda_arm" params="arm_id:='$(arg arm_id)' description_pkg:='franka_description_mti' connected_to:='' xyz:='0 0 0' rpy:='0 0 0' safety_distance:=0">
     <xacro:unless value="${not connected_to}">
       <joint name="${arm_id}_joint_${connected_to}" type="fixed">
